Commit message: fixed joint limits

File: sim/Fenrir.urdf (robot description, URDF)
Before this commit: robot Fenrir, 21 links, 20 joints
Links:
- removed link joint_four_bearing1
Joints:
- removed joint Rigid_13
- joint j1: limit lower=-1.570796 upper=1.570796 effort=100 velocity=100 -> lower=1.570796 upper=-1.570796 effort=100 velocity=100
- joint j3: limit lower=-1.570796 upper=1.570796 effort=100 velocity=100 -> lower=0.0 upper=3.141593 effort=100 velocity=100
- joint j5: limit lower=-1.570796 upper=1.570796 effort=100 velocity=100 -> lower=0.0 upper=3.141593 effort=100 velocity=100

Commit message: fixed simulation orientation

File: sim/Fenrir.urdf (robot description, URDF)
Before this commit: robot Fenrir, 20 links, 19 joints
Links:
- added link sim_pointer1, mass 0.0013428188019054788; collision mesh filename=meshes/sim_pointer1.stl scale=0.001 0.001 0.001; visual mesh filename=meshes/sim_pointer1.stl scale=0.001 0.001 0.001
Joints:
- added joint asim_joint: type fixed, parent gripper_body1, child sim_pointer1, origin xyz=-0.020744 0.016825 0.005144 rpy=1.57 0.15 -0.71
- joint j1: axis -0.029134 0.999576 0.0 -> -0.029134 -0.999576 0.0; limit lower=1.570796 upper=-1.570796 effort=100 velocity=100 -> lower=-1.570796 upper=1.570796 effort=100 velocity=100
